Commit message: fix: rename URDF joints to match deploy convention (R_hip_pitch etc)
URDF had Onshape names (right_hip_pitch_04), CAN publishes R_hip_pitch.
robot_state_publisher couldn't match /joint_states to URDF joints,
so all TF transforms stayed at origin.

File: deploy/biped_ws/src/biped_description/urdf/robot.urdf (robot description, URDF)
Before this commit: robot biped, 14 links, 13 joints
Joints:
- removed joint left_foot_pitch_02
- removed joint left_foot_roll_02
- removed joint left_hip_pitch_04
- removed joint left_hip_roll_03
- removed joint left_hip_yaw_03
- removed joint left_knee_04
- removed joint right_foot_pitch_02
- removed joint right_foot_roll_02
- removed joint right_hip_pitch_04
- removed joint right_hip_roll_03
- removed joint right_hip_yaw_03
- removed joint right_knee_04
- added joint L_foot_pitch: type revolute, parent kd_d_401l_6061, child arb_uj111_cross_bearing_2, origin xyz=-0.288552 0.0325676 0.05 rpy=0 0 3.14159, axis 0 0 1, limit lower=-0.872665 upper=0.523599 effort=30 velocity=10
- added joint L_foot_roll: type revolute, parent arb_uj111_cross_bearing_2, child foot_6061_2, origin xyz=0 0.03 -0.03 rpy=-1.5708 -1.5708 0, axis 0 0 1, limit lower=-0.261799 upper=0.261799 effort=30 velocity=10
- added joint L_hip_pitch: type revolute, parent assy_formfg___kd_b_102b_torso_btm, child kd_d_102l_6061, origin xyz=-0.000358761 0.0552809 -0.0828599 rpy=1.5708 0 -0, axis 0 0 1, limit lower=-1.0472 upper=2.21657 effort=100 velocity=10
- added joint L_hip_roll: type revolute, parent kd_d_102l_6061, child rs03, origin xyz=0.02925 -0.03 -0.071 rpy=3.14159 -1.5708 0, axis 0 0 1, limit lower=-0.20944 upper=2.26893 effort=50 velocity=10
- added joint L_hip_yaw: type revolute, parent rs03, child kd_d_301l_6061, origin xyz=0 0.142 -0.02525 rpy=1.5708 0 -0, axis 0 0 1, limit lower=-1.5708 upper=1.5708 effort=50 velocity=10
- added joint L_knee: type revolute, parent kd_d_301l_6061, child kd_d_401l_6061, origin xyz=0.02 -0.021 -0.212 rpy=0 -1.5708 0, axis 0 0 1, limit lower=0 upper=2.70526 effort=100 velocity=10
- added joint R_foot_pitch: type revolute, parent kd_d_401r_6061, child arb_uj111_cross_bearing, origin xyz=0.288552 -0.0326806 0.008 rpy=0 0 -0, axis 0 0 1, limit lower=-0.872665 upper=0.523599 effort=30 velocity=10
- added joint R_foot_roll: type revolute, parent arb_uj111_cross_bearing, child foot_6061, origin xyz=-0 0.03 -0.03 rpy=-1.5708 -1.5708 0, axis 0 0 1, limit lower=-0.261799 upper=0.261799 effort=30 velocity=10
- added joint R_hip_pitch: type revolute, parent assy_formfg___kd_b_102b_torso_btm, child kd_d_102r_6061, origin xyz=-0.000358761 -0.0547191 -0.0828599 rpy=1.5708 0 3.14159, axis 0 0 1, limit lower=-2.21657 upper=1.0472 effort=100 velocity=10
- added joint R_hip_roll: type revolute, parent kd_d_102r_6061, child kd_d_201r_6061, origin xyz=-0.02925 -0.03 -0.071 rpy=-0 -1.5708 0, axis 0 0 1, limit lower=-2.26893 upper=0.20944 effort=50 velocity=10
- added joint R_hip_yaw: type revolute, parent kd_d_201r_6061, child kd_d_301r_6061, origin xyz=-0 -0.142 -0.02525 rpy=-1.5708 -0 -0, axis 0 0 1, limit lower=-1.5708 upper=1.5708 effort=50 velocity=10
- added joint R_knee: type revolute, parent kd_d_301r_6061, child kd_d_401r_6061, origin xyz=0.022 0.021 -0.212 rpy=-0 1.5708 0, axis 0 0 1, limit lower=0 upper=2.70526 effort=100 velocity=10

Commit message: fix: rename URDF links from Onshape part names to semantic names
Onshape names (kd_d_401r_6061, arb_uj111_cross_bearing) →
semantic (base_link, R_knee_link, L_foot_pitch_link, etc.)
Enables proper TF tree with base_link as root for visualization.

File: deploy/biped_ws/src/biped_description/urdf/robot.urdf (robot description, URDF)
Before this commit: robot biped, 14 links, 13 joints
Links:
- removed link arb_uj111_cross_bearing
- removed link arb_uj111_cross_bearing_2
- removed link assy_formfg___kd_b_102b_torso_btm
- removed link foot_6061
- removed link foot_6061_2
- removed link kd_d_102l_6061
- removed link kd_d_102r_6061
- removed link kd_d_201r_6061
- removed link kd_d_301l_6061
- removed link kd_d_301r_6061
- removed link kd_d_401l_6061
- removed link kd_d_401r_6061
- removed link rs03
- added link L_foot_pitch_link, mass 0.317576; collision mesh filename=package://biped_description/meshes/arb_uj111_cross_bearing.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; visual mesh filename=package://biped_description/meshes/arb_uj111_cross_bearing.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
- added link L_foot_roll_link, mass 0.163562; collision mesh filename=package://biped_description/meshes/foot_6061.stl; visual mesh filename=package://biped_description/meshes/foot_6061.stl
- added link L_hip_pitch_link, mass 0.200236; collision mesh filename=package://biped_description/meshes/L_hip_pitch_link.stl; collision mesh filename=package://biped_description/meshes/kd_d_103l_6061.stl
- added link L_hip_roll_link, mass 2.04069; collision mesh filename=package://biped_description/meshes/ball_bearing_37x25x7.stl; collision mesh filename=package://biped_description/meshes/kd_d_201l_6061.stl
- added link L_hip_yaw_link, mass 1.82623; collision mesh filename=package://biped_description/meshes/L_hip_yaw_link.stl; collision mesh filename=package://biped_description/meshes/ball_bearing_37x25x7.stl
- added link L_knee_link, mass 1.25679; collision mesh filename=package://biped_description/meshes/L_knee_link.stl; collision mesh filename=package://biped_description/meshes/kd_d_402l_6061.stl
- added link R_foot_pitch_link, mass 0.317576; collision mesh filename=package://biped_description/meshes/arb_uj111_cross_bearing.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; visual mesh filename=package://biped_description/meshes/arb_uj111_cross_bearing.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
- added link R_foot_roll_link, mass 0.163562; collision mesh filename=package://biped_description/meshes/foot_6061.stl; visual mesh filename=package://biped_description/meshes/foot_6061.stl
- added link R_hip_pitch_link, mass 0.200236; collision mesh filename=package://biped_description/meshes/R_hip_pitch_link.stl; collision mesh filename=package://biped_description/meshes/kd_d_103r_6061.stl
- added link R_hip_roll_link, mass 2.0407; collision mesh filename=package://biped_description/meshes/R_hip_roll_link.stl; collision mesh filename=package://biped_description/meshes/ball_bearing_37x25x7.stl
- added link R_hip_yaw_link, mass 1.82618; collision mesh filename=package://biped_description/meshes/R_hip_yaw_link.stl; collision mesh filename=package://biped_description/meshes/ball_bearing_37x25x7.stl
- added link R_knee_link, mass 1.25681; collision mesh filename=package://biped_description/meshes/R_knee_link.stl; collision mesh filename=package://biped_description/meshes/kd_d_402r_6061.stl
- added link base_link, mass 3.4392; collision mesh filename=package://biped_description/meshes/assy_formfg___kc_d_107l_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; collision mesh filename=package://biped_description/meshes/assy_formfg___kc_d_107r_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
Joints:
- joint L_foot_pitch: child arb_uj111_cross_bearing_2 -> L_foot_pitch_link; parent kd_d_401l_6061 -> L_knee_link
- joint L_foot_roll: child foot_6061_2 -> L_foot_roll_link; parent arb_uj111_cross_bearing_2 -> L_foot_pitch_link
- joint L_hip_pitch: child kd_d_102l_6061 -> L_hip_pitch_link; parent assy_formfg___kd_b_102b_torso_btm -> base_link
- joint L_hip_roll: child rs03 -> L_hip_roll_link; parent kd_d_102l_6061 -> L_hip_pitch_link
- joint L_hip_yaw: child kd_d_301l_6061 -> L_hip_yaw_link; parent rs03 -> L_hip_roll_link
- joint L_knee: child kd_d_401l_6061 -> L_knee_link; parent kd_d_301l_6061 -> L_hip_yaw_link
- joint R_foot_pitch: child arb_uj111_cross_bearing -> R_foot_pitch_link; parent kd_d_401r_6061 -> R_knee_link
- joint R_foot_roll: child foot_6061 -> R_foot_roll_link; parent arb_uj111_cross_bearing -> R_foot_pitch_link
- joint R_hip_pitch: child kd_d_102r_6061 -> R_hip_pitch_link; parent assy_formfg___kd_b_102b_torso_btm -> base_link
- joint R_hip_roll: child kd_d_201r_6061 -> R_hip_roll_link; parent kd_d_102r_6061 -> R_hip_pitch_link
- joint R_hip_yaw: child kd_d_301r_6061 -> R_hip_yaw_link; parent kd_d_201r_6061 -> R_hip_roll_link
- joint R_knee: child kd_d_401r_6061 -> R_knee_link; parent kd_d_301r_6061 -> R_hip_yaw_link
- joint torso_to_battery: parent assy_formfg___kd_b_102b_torso_btm -> base_link

Commit message: fix: proper URDF rename — joints+links only, mesh filenames untouched
Previous sed globally replaced part names including inside mesh
filename paths. Now uses Python XML parser to rename only:
- joint name= attributes
- link name= attributes
- parent/child link= attributes
Mesh filename references stay matching the actual STL files on disk.

File: deploy/biped_ws/src/biped_description/urdf/robot.urdf (robot description, URDF)
Before this commit: robot biped, 14 links, 13 joints
Links:
- link L_hip_pitch_link: geometry collision mesh filename=package://biped_description/meshes/kd_d_102l_6061.stl; collision mesh filename=package://biped_description/meshes/kd_d_103l_6061.stl
- link L_hip_yaw_link: geometry collision mesh filename=package://biped_description/meshes/ball_bearing_37x25x7.stl; collision mesh filename=package://biped_description/meshes/kd_d_301l_6061.stl
- link L_knee_link: geometry collision mesh filename=package://biped_description/meshes/kd_d_401l_6061.stl; collision mesh filename=package://biped_description/meshes/kd_d_402l_6061.stl
- link R_hip_pitch_link: geometry collision mesh filename=package://biped_description/meshes/kd_d_102r_6061.stl; collision mesh filename=package://biped_description/meshes/kd_d_103r_6061.stl
- link R_hip_roll_link: geometry collision mesh filename=package://biped_description/meshes/ball_bearing_37x25x7.stl; collision mesh filename=package://biped_description/meshes/kd_d_201r_6061.stl
- link R_hip_yaw_link: geometry collision mesh filename=package://biped_description/meshes/ball_bearing_37x25x7.stl; collision mesh filename=package://biped_description/meshes/kd_d_301r_6061.stl
- link R_knee_link: geometry collision mesh filename=package://biped_description/meshes/kd_d_401r_6061.stl; collision mesh filename=package://biped_description/meshes/kd_d_402r_6061.stl
- link base_link: geometry collision mesh filename=package://biped_description/meshes/assy_formfg___kc_d_107l_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; collision mesh filename=package://biped_description/meshes/assy_formfg___kc_d_107r_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
