Commit message: urdf: reduce battery_chest mass 10kg→1kg (heavy URDF now 21.7kg)

File: urdf/heavy/robot.urdf (robot description, URDF)
Before this commit: robot biped, 14 links, 13 joints
Links:
- link battery_chest: mass 10.0 -> 1.0

Commit message: fix: URDF velocity limits matched to hardware
RS04 (hip_pitch/knee): 10→21 rad/s
RS03 (hip_roll/yaw): 10→21 rad/s
RS02 (foot): 10→30 rad/s

PhysX enforces URDF velocity limits at the physics level,
overriding the actuator config. This caused 10 rad/s chattering
in all sysid tests.

File: urdf/heavy/robot.urdf (robot description, URDF)
Before this commit: robot biped, 14 links, 13 joints
Joints:
- joint left_foot_pitch_02: limit lower=-0.872665 upper=0.523599 effort=30 velocity=10 -> lower=-0.872665 upper=0.523599 effort=30 velocity=30
- joint left_foot_roll_02: limit lower=-0.261799 upper=0.261799 effort=30 velocity=10 -> lower=-0.261799 upper=0.261799 effort=30 velocity=30
- joint left_hip_pitch_04: limit lower=-1.0472 upper=2.21657 effort=100 velocity=10 -> lower=-1.0472 upper=2.21657 effort=100 velocity=21
- joint left_hip_roll_03: limit lower=-0.20944 upper=2.26893 effort=50 velocity=10 -> lower=-0.20944 upper=2.26893 effort=50 velocity=21
- joint left_hip_yaw_03: limit lower=-1.5708 upper=1.5708 effort=50 velocity=10 -> lower=-1.5708 upper=1.5708 effort=50 velocity=21
- joint left_knee_04: limit lower=0 upper=2.70526 effort=100 velocity=10 -> lower=0 upper=2.70526 effort=100 velocity=21
- joint right_foot_pitch_02: limit lower=-0.872665 upper=0.523599 effort=30 velocity=10 -> lower=-0.872665 upper=0.523599 effort=30 velocity=30
- joint right_foot_roll_02: limit lower=-0.261799 upper=0.261799 effort=30 velocity=10 -> lower=-0.261799 upper=0.261799 effort=30 velocity=30
- joint right_hip_pitch_04: limit lower=-2.21657 upper=1.0472 effort=100 velocity=10 -> lower=-2.21657 upper=1.0472 effort=100 velocity=21
- joint right_hip_roll_03: limit lower=-2.26893 upper=0.20944 effort=50 velocity=10 -> lower=-2.26893 upper=0.20944 effort=50 velocity=21
- joint right_hip_yaw_03: limit lower=-1.5708 upper=1.5708 effort=50 velocity=10 -> lower=-1.5708 upper=1.5708 effort=50 velocity=21
- joint right_knee_04: limit lower=0 upper=2.70526 effort=100 velocity=10 -> lower=0 upper=2.70526 effort=100 velocity=21

File: urdf/light/robot.urdf (robot description, URDF)
Before this commit: robot biped, 14 links, 13 joints
Joints:
- joint left_foot_pitch_02: limit lower=-0.872665 upper=0.523599 effort=30 velocity=10 -> lower=-0.872665 upper=0.523599 effort=30 velocity=30
- joint left_foot_roll_02: limit lower=-0.261799 upper=0.261799 effort=30 velocity=10 -> lower=-0.261799 upper=0.261799 effort=30 velocity=30
- joint left_hip_pitch_04: limit lower=-1.0472 upper=2.21657 effort=100 velocity=10 -> lower=-1.0472 upper=2.21657 effort=100 velocity=21
- joint left_hip_roll_03: limit lower=-0.20944 upper=2.26893 effort=50 velocity=10 -> lower=-0.20944 upper=2.26893 effort=50 velocity=21
- joint left_hip_yaw_03: limit lower=-1.5708 upper=1.5708 effort=50 velocity=10 -> lower=-1.5708 upper=1.5708 effort=50 velocity=21
- joint left_knee_04: limit lower=0 upper=2.70526 effort=100 velocity=10 -> lower=0 upper=2.70526 effort=100 velocity=21
- joint right_foot_pitch_02: limit lower=-0.872665 upper=0.523599 effort=30 velocity=10 -> lower=-0.872665 upper=0.523599 effort=30 velocity=30
- joint right_foot_roll_02: limit lower=-0.261799 upper=0.261799 effort=30 velocity=10 -> lower=-0.261799 upper=0.261799 effort=30 velocity=30
- joint right_hip_pitch_04: limit lower=-2.21657 upper=1.0472 effort=100 velocity=10 -> lower=-2.21657 upper=1.0472 effort=100 velocity=21
- joint right_hip_roll_03: limit lower=-2.26893 upper=0.20944 effort=50 velocity=10 -> lower=-2.26893 upper=0.20944 effort=50 velocity=21
- joint right_hip_yaw_03: limit lower=-1.5708 upper=1.5708 effort=50 velocity=10 -> lower=-1.5708 upper=1.5708 effort=50 velocity=21
- joint right_knee_04: limit lower=0 upper=2.70526 effort=100 velocity=10 -> lower=0 upper=2.70526 effort=100 velocity=21

Commit message: heavy URDF: battery 1.0kg→0.5kg, size+pos matched to light
Battery: 0.5kg, box 126×146×50mm, at z=0.0436 (same as light).
Was: 1.0kg, 126×146×200mm, at z=0.1263.

File: urdf/heavy/robot.urdf (robot description, URDF)
Before this commit: robot biped, 14 links, 13 joints
Links:
- link battery_chest: mass 1.0 -> 0.5; geometry collision box size=0.1260 0.1460 0.05; visual box size=0.1260 0.1460 0.05
Joints:
- joint torso_to_battery: origin xyz=0.0004 0.0006 0.1263 rpy=0 0 0 -> xyz=-0.0004 0.0003 0.0436 rpy=0 0 0
